Commit message: fixed apporach stage ok

File: arctos_description/urdf/arctos.urdf.xacro (robot description, xacro)
@@ -5,7 +5,6 @@
   <xacro:include filename="$(find arctos_description)/urdf/common_properties.xacro" />
   <xacro:include filename="$(find arctos_description)/urdf/joint_link.xacro" />
+  <xacro:include filename="$(find arctos_description)/urdf/arctos_gripper.xacro" />
   <xacro:include filename="$(find arctos_description)/urdf/arctos_arm.xacro" />
-  <xacro:include filename="$(find arctos_description)/urdf/arctos_gripper.xacro" />
-  <xacro:include filename="$(find arctos_description)/urdf/arctos.ros2_control.xacro" />
   <!--- from moveit config package  -->
   <!-- <xacro:include filename="$(find arctos_description)/urdf/arctos.ros2_control.xacro" /> -->
@@ -16,4 +15,5 @@
     <origin xyz="0.0 0.0 0.0" rpy="0 0 0"/>
   </joint>
+  <xacro:include filename="$(find arctos_description)/urdf/arctos.ros2_control.xacro" />
   <!-- ros2_control with mock components is included directly from arctos.ros2_control.xacro -->
   <!-- include gazebo parameters -->

File: arctos_description/urdf/arctos_arm.xacro (robot description, xacro)
@@ -7,5 +7,5 @@
     name="base_link"
     origin_xyz="0 0 0" origin_rpy="0 0 0"
-    material_name="green"
+    material_name="white"
     inertia_origin_xyz="0.0009375030874740357 0.047087016508753216 0.06663230338123677"
     inertia_origin_rpy="0 0 0"
@@ -66,11 +66,12 @@
   />
   <!-- Define all joints -->
-  <joint name="world_joint" type="fixed">
+  <joint name="base_joint" type="fixed">
     <parent link="world" />
     <child link="base_link" />
     <origin xyz="0 0 0" rpy="0 0 0" />
+    <axis xyz="0 0 1" />
   </joint>
   <xacro:arctos_joint
-    name="X_joint" type="revolute"
+    name="X_joint" type="continuous"
     parent="base_link" child="Link_1_1"
     origin_xyz="0.0 0.0 0.1126" origin_rpy="0 0 0"
@@ -79,5 +80,5 @@
   />
   <xacro:arctos_joint
-    name="Y_joint" type="revolute"
+    name="Y_joint" type="continuous"
     parent="Link_1_1" child="Link_2_1"
     origin_xyz="0.0 -0.020356 ${0.2876-0.1126}" origin_rpy="0 0 0"
@@ -86,5 +87,5 @@
   />
   <xacro:arctos_joint
-    name="Z_joint" type="revolute"
+    name="Z_joint" type="continuous"
     parent="Link_2_1" child="Link_3_1"
     origin_xyz="0.0 0.001365 0.261035" origin_rpy="0 0 0"
@@ -93,5 +94,5 @@
   />
   <xacro:arctos_joint
-    name="A_joint" type="revolute"
+    name="A_joint" type="continuous"
     parent="Link_3_1" child="Link_4_1"
     origin_xyz="0 -0.13881 0.0217651" origin_rpy="0 0 0"
@@ -100,5 +101,5 @@
   />
   <xacro:arctos_joint
-    name="B_joint" type="revolute"
+    name="B_joint" type="continuous"
     parent="Link_4_1" child="Link_5_1"
     origin_xyz="0.0 -0.12543 -0.00184" origin_rpy="0 0 0"
@@ -107,5 +108,5 @@
   />
   <xacro:arctos_joint
-    name="C_joint" type="revolute"
+    name="C_joint" type="continuous"
     parent="Link_5_1" child="Link_6_1"
     origin_xyz="0.0 -0.0398 0.0" origin_rpy="0 0 0"
@@ -117,5 +118,4 @@
     <child link="tool_link"/>
     <origin xyz="0.0 0.0 0.0" rpy="0 0 0"/>
-    <axis xyz="-0.0 1.0 -0.0"/>
   </joint>
   <!-- Activate Gazebo plugin -->

File: arctos_description/urdf/arctos_gripper.xacro (robot description, xacro)
@@ -2,5 +2,5 @@
 <robot xmlns:xacro="http://www.ros.org/wiki/xacro">
   <!-- <xacro:include filename="$(find arctos_description)/urdf/joint_link.xacro" /> -->
-  <!-- Arctos gripper base -->
+    <!-- Arctos Simple Pinch Gripper -->
   <xacro:arctos_link
     name="Gripper_1"
@@ -16,6 +16,6 @@
     material_name="white"
     inertia_origin_xyz="-0.0 -0.0211 0.0" inertia_origin_rpy="0 0 0"
-    mass="0.001"
-    ixx="1.4e-8" iyy="4.2e-8" izz="3.5e-8" ixy="0.0" iyz="0.0" ixz="0.0"
+    mass="0."
+    ixx="0.0" iyy="0.0" izz="0.0" ixy="-0.0" iyz="0.0" ixz="0.0"
   />
   <xacro:arctos_link
@@ -24,6 +24,6 @@
     material_name="white"
     inertia_origin_xyz="-0.001 -0.0211 0.0" inertia_origin_rpy="0 0 0"
-    mass="0.001"
-    ixx="1.4e-8" iyy="4.2e-8" izz="3.5e-8" ixy="0.0" iyz="0.0" ixz="0.0"
+    mass="0."
+    ixx="0.0" iyy="0.0" izz="0.0" ixy="-0.0" iyz="0.0" ixz="0.0"
   />
   <!-- Fixed gripper joint, no axis needed -->
@@ -35,4 +35,17 @@
   /> -->
   <!-- Left jaw joint, prismatic with axis directly defined -->
+  <xacro:arctos_joint
+    name="Left_jaw_joint"
+    type="prismatic"
+    parent="Gripper_1"
+    child="Left_jaw_1"
+    origin_xyz="0.0 0.0 0.0"
+    origin_rpy="0 0 0"
+    axis_xyz="0 0 1"
+    limit_u="0.015"
+    limit_l="0.0"
+    limit_e="1.0"
+    limit_v="10.0"
+  />
   <xacro:arctos_joint
     name="Right_jaw_joint"
@@ -48,11 +61,3 @@
     limit_v="10.0"
   />
-  <joint name="Left_jaw_joint" type="prismatic">
-    <parent link="Gripper_1"/>
-    <child link="Left_jaw_1"/>
-    <origin xyz="0.0 0.0 0.0" rpy="0 0 0"/>
-    <axis xyz="0 0 1"/>
-    <mimic joint="Right_jaw_joint" multiplier="-1" offset="0.0"/>
-    <limit lower="-0.015" upper="0.0" effort="1.0" velocity="10.0" acceleration="5.0"/>
-  </joint>
 </robot>
