Commit message: left jaw mimic right jaw

File: arctos_description/urdf/arctos_gripper.xacro (robot description, xacro)
@@ -16,6 +16,6 @@
     material_name="white"
     inertia_origin_xyz="-0.0 -0.0211 0.0" inertia_origin_rpy="0 0 0"
-    mass="0."
-    ixx="0.0" iyy="0.0" izz="0.0" ixy="-0.0" iyz="0.0" ixz="0.0"
+    mass="0.001"
+    ixx="1.4e-8" iyy="4.2e-8" izz="3.5e-8" ixy="0.0" iyz="0.0" ixz="0.0"
   />
   <xacro:arctos_link
@@ -24,6 +24,6 @@
     material_name="white"
     inertia_origin_xyz="-0.001 -0.0211 0.0" inertia_origin_rpy="0 0 0"
-    mass="0."
-    ixx="0.0" iyy="0.0" izz="0.0" ixy="-0.0" iyz="0.0" ixz="0.0"
+    mass="0.001"
+    ixx="1.4e-8" iyy="4.2e-8" izz="3.5e-8" ixy="0.0" iyz="0.0" ixz="0.0"
   />
   <!-- Fixed gripper joint, no axis needed -->
@@ -35,17 +35,4 @@
   /> -->
   <!-- Left jaw joint, prismatic with axis directly defined -->
-  <xacro:arctos_joint
-    name="Left_jaw_joint"
-    type="prismatic"
-    parent="Gripper_1"
-    child="Left_jaw_1"
-    origin_xyz="0.0 0.0 0.0"
-    origin_rpy="0 0 0"
-    axis_xyz="0 0 1"
-    limit_u="0.015"
-    limit_l="0.0"
-    limit_e="1.0"
-    limit_v="10.0"
-  />
   <xacro:arctos_joint
     name="Right_jaw_joint"
@@ -61,3 +48,11 @@
     limit_v="10.0"
   />
+   <joint name="Left_jaw_joint" type="prismatic">
+    <parent link="Gripper_1"/>
+    <child link="Left_jaw_1"/>
+    <origin xyz="0.0 0.0 0.0" rpy="0 0 0"/>
+    <axis xyz="0 0 1"/>
+    <mimic joint="Right_jaw_joint" multiplier="-1" offset="0.0"/>
+    <limit lower="-0.015" upper="0.0" effort="1.0" velocity="10.0"/>
+  </joint>
 </robot>
