Commit message: FIX: should be left  mimic right jaw. 3 changes needed: controllers.yaml, moveit_controllers.yaml, and srd file for close and open value, which can be tested/get from moveit2 motion plan

File: arctos_description/urdf/arctos.ros2_control.xacro (robot description, xacro)
@@ -42,8 +42,8 @@
         </state_interface>
     </joint>
-    <joint name="Left_jaw_joint">
+    <joint name="Right_jaw_joint">
         <command_interface name="position"/>
         <state_interface name="position">
-          <param name="initial_value">0.0</param>
+          <!-- <param name="initial_value">0.0</param> -->
         </state_interface>
     </joint>

File: arctos_description/urdf/arctos_gripper.xacro (robot description, xacro)
@@ -36,8 +36,8 @@
   <!-- Left jaw joint, prismatic with axis directly defined -->
   <xacro:arctos_joint
-    name="Left_jaw_joint"
+    name="Right_jaw_joint"
     type="prismatic"
     parent="Gripper_1"
-    child="Left_jaw_1"
+    child="Right_jaw_1"
     origin_xyz="0.0 0.0 0.0"
     origin_rpy="0 0 0"
@@ -48,10 +48,10 @@
     limit_v="10.0"
   />
-  <joint name="Right_jaw_joint" type="prismatic">
+  <joint name="Left_jaw_joint" type="prismatic">
     <parent link="Gripper_1"/>
-    <child link="Right_jaw_1"/>
+    <child link="Left_jaw_1"/>
     <origin xyz="0.0 0.0 0.0" rpy="0 0 0"/>
     <axis xyz="0 0 1"/>
-    <mimic joint="Left_jaw_joint" multiplier="-1" offset="0.0"/>
+    <mimic joint="Right_jaw_joint" multiplier="-1" offset="0.0"/>
     <limit lower="-0.015" upper="0.0" effort="1.0" velocity="10.0"/>
   </joint>

Commit message: switch to use servo_can.hpp for can drive for simplicity. can move but incorrect position.

File: arctos_description/urdf/arctos.ros2_control.xacro (robot description, xacro)
@@ -1,61 +1,33 @@
 <?xml version="1.0"?>
 <robot xmlns:xacro="http://www.ros.org/wiki/xacro">
+  <xacro:macro name="arctos_joint" params="name can_id gear_ratio">
+    <joint name="${name}">
+      <param name='can_id'>${can_id}</param>
+      <param name='gear_ratio'>${gear_ratio}</param>
+      <command_interface name="position"/>
+      <state_interface name="position">
+        <param name="initial_value">0.0</param>
+      </state_interface>
+      <state_interface name="velocity">
+        <param name="initial_value">0.0</param>
+      </state_interface>
+      <!-- <state_interface name="effort">
+        <param name="initial_value">0.0</param>
+      </state_interface> -->
+    </joint>
+  </xacro:macro>
   <ros2_control name="arm" type="system">
     <hardware>
-      <!-- By default, set up controllers for simulation. This won't work on real hardware -->
-      <!-- <plugin>mock_components/GenericSystem</plugin> -->
       <plugin>arctos_hardware_interface/ArctosHardwareInterface</plugin>
       <param name='can_interface'>can0</param>
-      <param name='gear_ratio_X'>13.5</param>
-      <param name='gear_ratio_Y'>150.0</param>
-      <param name='gear_ratio_Z'>150.0</param>
-      <param name='gear_ratio_A'>48.0</param>
-      <param name='gear_ratio_B'>67.82</param>
-      <param name='gear_ratio_C'>67.82</param>
       <param name='accel'>10</param>
       <param name='vel'>100</param>
-      <param name='can_id_X'>1</param>
-      <param name='can_id_Y'>2</param>
-      <param name='can_id_Z'>3</param>
-      <param name='can_id_A'>4</param>
-      <param name='can_id_B'>5</param>
-      <param name='can_id_C'>6</param>
     </hardware>
-    <joint name="X_joint">
-        <command_interface name="position"/>
-        <state_interface name="position">
-          <param name="initial_value">0.0</param>
-        </state_interface>
-    </joint>
-    <joint name="Y_joint">
-        <command_interface name="position"/>
-        <state_interface name="position">
-          <param name="initial_value">0.0</param>
-        </state_interface>
-    </joint>
-    <joint name="Z_joint">
-        <command_interface name="position"/>
-        <state_interface name="position">
-          <param name="initial_value">0.0</param>
-        </state_interface>
-    </joint>
-    <joint name="A_joint">
-        <command_interface name="position"/>
-        <state_interface name="position">
-          <param name="initial_value">0.0</param>
-        </state_interface>
-    </joint>
-    <joint name="B_joint">
-        <command_interface name="position"/>
-        <state_interface name="position">
-          <param name="initial_value">0.0</param>
-        </state_interface>
-    </joint>
-    <joint name="C_joint">
-        <command_interface name="position"/>
-        <state_interface name="position">
-          <param name="initial_value">0.0</param>
-        </state_interface>
-    </joint>
+    <xacro:arctos_joint name="X_joint" can_id="1" gear_ratio="13.5"/>
+    <xacro:arctos_joint name="Y_joint" can_id="2" gear_ratio="150.0"/>
+    <xacro:arctos_joint name="Z_joint" can_id="3" gear_ratio="150.0"/>
+    <xacro:arctos_joint name="A_joint" can_id="4" gear_ratio="48.0"/>
+    <xacro:arctos_joint name="B_joint" can_id="5" gear_ratio="67.82"/>
+    <xacro:arctos_joint name="C_joint" can_id="6" gear_ratio="67.82"/>
   </ros2_control>
   <ros2_control name="gripper" type="system">
@@ -70,3 +42,3 @@
     </joint>
   </ros2_control>
-</robot>
+  </robot>

Commit message: ADD: add mtc_tutorial pkg, add world link for moveit2

File: arctos_description/urdf/arctos.ros2_control.xacro (robot description, xacro)
@@ -17,10 +17,17 @@
     </joint>
   </xacro:macro>
+  <xacro:arg name="use_fake_hardware" default="true"/>
   <ros2_control name="arm" type="system">
     <hardware>
-      <plugin>arctos_hardware_interface/ArctosHardwareInterface</plugin>
-      <param name='can_interface'>can0</param>
-      <param name='accel'>10</param>
-      <param name='vel'>100</param>
+      <xacro:if value="$(arg use_fake_hardware)">
+        <plugin>mock_components/GenericSystem</plugin>
+      </xacro:if>
+      <xacro:unless value="$(arg use_fake_hardware)">
+        <plugin>mock_components/GenericSystem</plugin>
+        <!-- <plugin>arctos_hardware_interface/ArctosHardwareInterface</plugin> -->
+        <param name='can_interface'>can0</param>
+        <param name='accel'>10</param>
+        <param name='vel'>100</param>
+      </xacro:unless>
     </hardware>
     <xacro:arctos_joint name="X_joint" can_id="1" gear_ratio="13.5"/>

File: arctos_description/urdf/arctos_arm.xacro (robot description, xacro)
@@ -2,5 +2,5 @@
 <robot xmlns:xacro="http://www.ros.org/wiki/xacro">
   <!-- Define all links -->
-  <!-- <link name="world" /> -->
+  <link name="world" />
   <link name="tool_link" />
   <xacro:arctos_link
@@ -66,10 +66,9 @@
   />
   <!-- Define all joints -->
-  <!-- <joint name="base_joint" type="fixed">
+  <joint name="world_joint" type="fixed">
     <parent link="world" />
     <child link="base_link" />
     <origin xyz="0 0 0" rpy="0 0 0" />
-    <axis xyz="0 0 1" />
-  </joint> -->
+  </joint>
   <xacro:arctos_joint
     name="X_joint" type="revolute"

File: arctos_description/urdf/arctos_gripper.xacro (robot description, xacro)
@@ -54,5 +54,5 @@
     <axis xyz="0 0 1"/>
     <mimic joint="Right_jaw_joint" multiplier="-1" offset="0.0"/>
-    <limit lower="-0.015" upper="0.0" effort="1.0" velocity="10.0"/>
+    <limit lower="-0.015" upper="0.0" effort="1.0" velocity="10.0" acceleration="5.0"/>
   </joint>
 </robot>

Commit message: FIX: launch file,  use_fake_hardware arg, xml

File: arctos_description/urdf/arctos.ros2_control.xacro (robot description, xacro)
@@ -1,8 +1,11 @@
 <?xml version="1.0"?>
 <robot xmlns:xacro="http://www.ros.org/wiki/xacro">
+  <!-- ARGUMENT TO TOGGLE FAKE HARDWARE -->
+  <xacro:arg name="use_fake_hardware" default="false"/>
+  <!-- JOINT MACRO -->
   <xacro:macro name="arctos_joint" params="name can_id gear_ratio">
     <joint name="${name}">
-      <param name='can_id'>${can_id}</param>
-      <param name='gear_ratio'>${gear_ratio}</param>
+      <param name="can_id">${can_id}</param>
+      <param name="gear_ratio">${gear_ratio}</param>
       <command_interface name="position"/>
       <state_interface name="position">
@@ -12,40 +15,42 @@
         <param name="initial_value">0.0</param>
       </state_interface>
-      <!-- <state_interface name="effort">
-        <param name="initial_value">0.0</param>
-      </state_interface> -->
     </joint>
   </xacro:macro>
-  <xacro:arg name="use_fake_hardware" default="true"/>
-  <ros2_control name="arm" type="system">
-    <hardware>
-      <xacro:if value="$(arg use_fake_hardware)">
+  <!-- ROS2 CONTROL MACRO -->
+  <xacro:macro name="arctos_ros2_control" params="use_fake_hardware:=false">
+    <ros2_control name="arm" type="system">
+      <hardware>
+        <xacro:if value="$(arg use_fake_hardware)">
+          <plugin>mock_components/GenericSystem</plugin>
+        </xacro:if>
+        <xacro:unless value="$(arg use_fake_hardware)">
+          <plugin>arctos_hardware_interface/ArctosHardwareInterface</plugin>
+          <class_type>arctos_hardware_interface::ArctosHardwareInterface</class_type>
+          <param name="can_interface">can0</param>
+          <param name="accel">10</param>
+          <param name="vel">100</param>
+        </xacro:unless>
+      </hardware>
+      <!-- JOINT DEFINITIONS -->
+      <xacro:arctos_joint name="X_joint" can_id="1" gear_ratio="13.5"/>
+      <xacro:arctos_joint name="Y_joint" can_id="2" gear_ratio="150.0"/>
+      <xacro:arctos_joint name="Z_joint" can_id="3" gear_ratio="150.0"/>
+      <xacro:arctos_joint name="A_joint" can_id="4" gear_ratio="48.0"/>
+      <xacro:arctos_joint name="B_joint" can_id="5" gear_ratio="67.82"/>
+      <xacro:arctos_joint name="C_joint" can_id="6" gear_ratio="67.82"/>
+    </ros2_control>
+    <ros2_control name="gripper" type="system">
+      <hardware>
         <plugin>mock_components/GenericSystem</plugin>
-      </xacro:if>
-      <xacro:unless value="$(arg use_fake_hardware)">
-        <plugin>mock_components/GenericSystem</plugin>
-        <!-- <plugin>arctos_hardware_interface/ArctosHardwareInterface</plugin> -->
-        <param name='can_interface'>can0</param>
-        <param name='accel'>10</param>
-        <param name='vel'>100</param>
-      </xacro:unless>
-    </hardware>
-    <xacro:arctos_joint name="X_joint" can_id="1" gear_ratio="13.5"/>
-    <xacro:arctos_joint name="Y_joint" can_id="2" gear_ratio="150.0"/>
-    <xacro:arctos_joint name="Z_joint" can_id="3" gear_ratio="150.0"/>
-    <xacro:arctos_joint name="A_joint" can_id="4" gear_ratio="48.0"/>
-    <xacro:arctos_joint name="B_joint" can_id="5" gear_ratio="67.82"/>
-    <xacro:arctos_joint name="C_joint" can_id="6" gear_ratio="67.82"/>
-  </ros2_control>
-  <ros2_control name="gripper" type="system">
-    <hardware>
-      <plugin>mock_components/GenericSystem</plugin>
-    </hardware>
-    <joint name="Right_jaw_joint">
-      <command_interface name="position"/>
-      <state_interface name="position">
-        <param name="initial_value">0.0</param>
-      </state_interface>
-    </joint>
-  </ros2_control>
-  </robot>
+      </hardware>
+      <joint name="Right_jaw_joint">
+        <command_interface name="position"/>
+        <state_interface name="position">
+          <param name="initial_value">0.0</param>
+        </state_interface>
+      </joint>
+    </ros2_control>
+  </xacro:macro>
+  <!-- INSTANTIATE THE MACRO -->
+  <xacro:arctos_ros2_control use_fake_hardware="$(arg use_fake_hardware)"/>
+</robot>

Commit message: amend: rm gripper_base_joint off srdf, add gripper in h/w interface, add state vel for gripper in urdf"

File: arctos_description/urdf/arctos.ros2_control.xacro (robot description, xacro)
@@ -39,15 +39,22 @@
       <xacro:arctos_joint name="B_joint" can_id="5" gear_ratio="67.82"/>
       <xacro:arctos_joint name="C_joint" can_id="6" gear_ratio="67.82"/>
-    </ros2_control>
+      <xacro:arctos_joint name="Right_jaw_joint" can_id="7" gear_ratio="1"/>
+    <!-- </ros2_control>
     <ros2_control name="gripper" type="system">
       <hardware>
         <plugin>mock_components/GenericSystem</plugin>
-      </hardware>
-      <joint name="Right_jaw_joint">
+      </hardware> -->
+      <!-- <joint name="Right_jaw_joint">
         <command_interface name="position"/>
         <state_interface name="position">
           <param name="initial_value">0.0</param>
         </state_interface>
-      </joint>
+        <state_interface name="velocity">
+          <param name="initial_value">0.0</param>
+        </state_interface>
+        <state_interface name="effort">
+          <param name="initial_value">0.0</param>
+        </state_interface>
+      </joint> -->
     </ros2_control>
   </xacro:macro>

Commit message: amend single src of min & max pos for urdf, and get the params in h/w int for clamp cmd in write, inc acc_ by 10 to 20.

File: arctos_description/urdf/arctos.ros2_control.xacro (robot description, xacro)
@@ -4,9 +4,12 @@
   <xacro:arg name="use_fake_hardware" default="false"/>
   <!-- JOINT MACRO -->
-  <xacro:macro name="arctos_joint" params="name can_id gear_ratio">
+  <xacro:macro name="arctos_joint" params="name can_id gear_ratio limit_l limit_u" >
     <joint name="${name}">
       <param name="can_id">${can_id}</param>
       <param name="gear_ratio">${gear_ratio}</param>
-      <command_interface name="position"/>
+      <command_interface name="position">
+        <param name="min">${limit_l}</param>
+        <param name="max">${limit_u}</param>
+      </command_interface>
       <state_interface name="position">
         <param name="initial_value">0.0</param>
@@ -28,16 +31,17 @@
           <class_type>arctos_hardware_interface::ArctosHardwareInterface</class_type>
           <param name="can_interface">can0</param>
-          <param name="accel">10</param>
+          <param name="accel">20</param>
           <param name="vel">100</param>
         </xacro:unless>
       </hardware>
       <!-- JOINT DEFINITIONS -->
-      <xacro:arctos_joint name="X_joint" can_id="1" gear_ratio="13.5"/>
-      <xacro:arctos_joint name="Y_joint" can_id="2" gear_ratio="-150.0"/>
-      <xacro:arctos_joint name="Z_joint" can_id="3" gear_ratio="150.0"/>
-      <xacro:arctos_joint name="A_joint" can_id="4" gear_ratio="48.0"/>
-      <xacro:arctos_joint name="B_joint" can_id="5" gear_ratio="67.82"/>
-      <xacro:arctos_joint name="C_joint" can_id="6" gear_ratio="67.82"/>
-      <xacro:arctos_joint name="Right_jaw_joint" can_id="7" gear_ratio="1"/>
+      <xacro:arctos_joint name="X_joint" can_id="1" gear_ratio="13.5" limit_l="${X_min_pos}" limit_u="${X_max_pos}"/>
+      <xacro:arctos_joint name="Y_joint" can_id="2" gear_ratio="-150.0" limit_l="${Y_min_pos}" limit_u="${Y_max_pos}"/>
+      <xacro:arctos_joint name="Z_joint" can_id="3" gear_ratio="150.0" limit_l="${Z_min_pos}" limit_u="${Z_max_pos}"/>
+      <xacro:arctos_joint name="A_joint" can_id="4" gear_ratio="48.0" limit_l="${A_min_pos}" limit_u="${A_max_pos}"/>
+      <xacro:arctos_joint name="B_joint" can_id="5" gear_ratio="67.82" limit_l="${B_min_pos}" limit_u="${B_max_pos}"/>
+      <xacro:arctos_joint name="C_joint" can_id="6" gear_ratio="67.82" limit_l="${C_min_pos}" limit_u="${C_max_pos}"/>
+      <xacro:arctos_joint name="Right_jaw_joint" can_id="7" gear_ratio="1" limit_l="0.0"
+      limit_u="0.015"/>
     <!-- </ros2_control>
     <ros2_control name="gripper" type="system">

File: arctos_description/urdf/arctos.urdf.xacro (robot description, xacro)
@@ -3,4 +3,16 @@
   <xacro:arg name='is_sim' default='true' />
   <xacro:arg name="use_fake_hardware" default="false" />
+  <xacro:property name="X_max_pos" value="${pi}"/>
+  <xacro:property name="X_min_pos" value="${-pi}"/>
+  <xacro:property name="Y_max_pos" value="2.18"/>
+  <xacro:property name="Y_min_pos" value="-0.96"/>
+  <xacro:property name="Z_max_pos" value="${70/180*pi}"/>
+  <xacro:property name="Z_min_pos" value="${-pi/2}"/>
+  <xacro:property name="A_max_pos" value="${pi}"/>
+  <xacro:property name="A_min_pos" value="${-pi}"/>
+  <xacro:property name="B_max_pos" value="${1.55}"/>
+  <xacro:property name="B_min_pos" value="${-1.55}"/>
+  <xacro:property name="C_max_pos" value="${pi}"/>
+  <xacro:property name="C_min_pos" value="${-pi}"/>
   <xacro:include filename="$(find arctos_description)/urdf/common_properties.xacro" />
   <xacro:include filename="$(find arctos_description)/urdf/joint_link.xacro" />

File: arctos_description/urdf/arctos_arm.xacro (robot description, xacro)
@@ -77,5 +77,5 @@
     origin_xyz="0.0 0.0 0.1126" origin_rpy="0 0 0"
     axis_xyz="-0.0 0.0 1.0"
-    limit_u="${pi}" limit_l="${-pi}" limit_e="24.3" limit_v="15.0"
+    limit_u="${X_max_pos}" limit_l="${X_min_pos}" limit_e="24.3" limit_v="15.0"
   />
   <xacro:arctos_joint
@@ -84,5 +84,5 @@
     origin_xyz="0.0 -0.020356 ${0.2876-0.1126}" origin_rpy="0 0 0"
     axis_xyz="1.0 -0.0 -0.0"
-    limit_u="2.18" limit_l="-0.96" limit_e="270.0" limit_v="1.4"
+    limit_u="${Y_max_pos}" limit_l="${Y_min_pos}" limit_e="270.0" limit_v="1.4"
   />
   <xacro:arctos_joint
@@ -91,5 +91,5 @@
     origin_xyz="0.0 0.001365 0.261035" origin_rpy="0 0 0"
     axis_xyz="1.0 -0.0 0.0"
-    limit_u="${70/180*pi}" limit_l="${-pi/2}" limit_e="97.0" limit_v="1.4"
+    limit_u="${Z_max_pos}" limit_l="${Z_min_pos}" limit_e="97.0" limit_v="1.4"
   />
   <xacro:arctos_joint
@@ -98,5 +98,5 @@
     origin_xyz="0 -0.13881 0.0217651" origin_rpy="0 0 0"
     axis_xyz="-0.0 1.0 -0.0"
-    limit_u="${pi}" limit_l="${-pi}" limit_e="22.0" limit_v="4.4"
+    limit_u="${A_max_pos}" limit_l="${A_min_pos}" limit_e="22.0" limit_v="4.4"
   />
   <xacro:arctos_joint
@@ -105,5 +105,5 @@
     origin_xyz="0.0 -0.12543 -0.00184" origin_rpy="0 0 0"
     axis_xyz="-1.0 -0.0 0.0"
-    limit_u="1.55" limit_l="-1.55" limit_e="16.0" limit_v="3.0"
+    limit_u="${B_max_pos}" limit_l="${B_min_pos}" limit_e="16.0" limit_v="3.0"
   />
   <xacro:arctos_joint
@@ -112,5 +112,5 @@
     origin_xyz="0.0 -0.0398 0.0" origin_rpy="0 0 0"
     axis_xyz="-0.0 1.0 -0.0"
-    limit_u="${pi}" limit_l="${-pi}" limit_e="16.0" limit_v="3.0"
+    limit_u="${C_max_pos}" limit_l="${C_min_pos}" limit_e="16.0" limit_v="3.0"
   />
   <joint name ="hand_tool_joint" type="fixed">

Commit message: amend: handle differential gearbox in on_active

File: arctos_description/urdf/arctos.ros2_control.xacro (robot description, xacro)
@@ -41,5 +41,5 @@
       <xacro:arctos_joint name="A_joint" can_id="4" gear_ratio="48.0" limit_l="${A_min_pos}" limit_u="${A_max_pos}"/>
       <xacro:arctos_joint name="B_joint" can_id="5" gear_ratio="67.82" limit_l="${B_min_pos}" limit_u="${B_max_pos}"/>
-      <xacro:arctos_joint name="C_joint" can_id="6" gear_ratio="-67.82" limit_l="${C_min_pos}" limit_u="${C_max_pos}"/>
+      <xacro:arctos_joint name="C_joint" can_id="6" gear_ratio="67.82" limit_l="${C_min_pos}" limit_u="${C_max_pos}"/>
       <xacro:arctos_joint name="Right_jaw_joint" can_id="7" gear_ratio="1" limit_l="0.0"
       limit_u="0.015"/>

File: arctos_description/urdf/arctos_arm.xacro (robot description, xacro)
@@ -15,5 +15,5 @@
   <xacro:arctos_link
     name="Link_1_1"
-    origin_xyz="-0.0 -0.000 -0.1126" origin_rpy="0 0 0"
+    origin_xyz="-0.0 0.0 -0.1126" origin_rpy="0 0 0"
     material_name="white"
     inertia_origin_xyz="-0.0088 -0.0005 ${0.2116-0.1126}" inertia_origin_rpy="0 0 0"
@@ -61,7 +61,7 @@
     origin_xyz="0.0 0.323 -0.5685" origin_rpy="0 0 0"
     material_name="white"
-    inertia_origin_xyz="-0.0 -0.0 0.0" inertia_origin_rpy="0.0 0.0 0.0"
+    inertia_origin_xyz="0.0 0.0 0.0" inertia_origin_rpy="0.0 0.0 0.0"
     mass="1e-3"
-    ixx="1e-3" iyy="1e-3" izz="1e-3" ixy="-0.0" iyz="0.0" ixz="0.0"
+    ixx="1e-3" iyy="1e-3" izz="1e-3" ixy="0.0" iyz="0.0" ixz="0.0"
   />
   <!-- Define all joints -->
@@ -76,5 +76,5 @@
     parent="base_link" child="Link_1_1"
     origin_xyz="0.0 0.0 0.1126" origin_rpy="0 0 0"
-    axis_xyz="-0.0 0.0 1.0"
+    axis_xyz="0 0 1"
     limit_u="${X_max_pos}" limit_l="${X_min_pos}" limit_e="24.3" limit_v="15.0"
   />
@@ -83,5 +83,5 @@
     parent="Link_1_1" child="Link_2_1"
     origin_xyz="0.0 -0.020356 ${0.2876-0.1126}" origin_rpy="0 0 0"
-    axis_xyz="1.0 -0.0 -0.0"
+    axis_xyz="1 0 0"
     limit_u="${Y_max_pos}" limit_l="${Y_min_pos}" limit_e="270.0" limit_v="1.4"
   />
@@ -90,5 +90,5 @@
     parent="Link_2_1" child="Link_3_1"
     origin_xyz="0.0 0.001365 0.261035" origin_rpy="0 0 0"
-    axis_xyz="1.0 -0.0 0.0"
+    axis_xyz="1 0 0"
     limit_u="${Z_max_pos}" limit_l="${Z_min_pos}" limit_e="97.0" limit_v="1.4"
   />
@@ -97,5 +97,5 @@
     parent="Link_3_1" child="Link_4_1"
     origin_xyz="0 -0.13881 0.0217651" origin_rpy="0 0 0"
-    axis_xyz="-0.0 1.0 -0.0"
+    axis_xyz="0 1 0"
     limit_u="${A_max_pos}" limit_l="${A_min_pos}" limit_e="22.0" limit_v="4.4"
   />
@@ -104,5 +104,5 @@
     parent="Link_4_1" child="Link_5_1"
     origin_xyz="0.0 -0.12543 -0.00184" origin_rpy="0 0 0"
-    axis_xyz="-1.0 -0.0 0.0"
+    axis_xyz="1 0 0"
     limit_u="${B_max_pos}" limit_l="${B_min_pos}" limit_e="16.0" limit_v="3.0"
   />
@@ -111,5 +111,5 @@
     parent="Link_5_1" child="Link_6_1"
     origin_xyz="0.0 -0.0398 0.0" origin_rpy="0 0 0"
-    axis_xyz="-0.0 1.0 -0.0"
+    axis_xyz="0 1 0"
     limit_u="${C_max_pos}" limit_l="${C_min_pos}" limit_e="16.0" limit_v="3.0"
   />
@@ -117,5 +117,5 @@
     <parent link="Link_6_1"/>
     <child link="tool_link"/>
-    <origin xyz="0.0 0.0 0.0" rpy="0 0 0"/>
+    <origin xyz="0 0 0" rpy="0 0 0"/>
   </joint>
   <!-- Activate Gazebo plugin -->
