Commit message: amend: diff vel, acc for motors (in joint_limit & h/w int& xacro). base slowest.

File: arctos_description/urdf/arctos.ros2_control.xacro (robot description, xacro)
@@ -4,7 +4,9 @@
   <xacro:arg name="use_fake_hardware" default="false"/>
   <!-- JOINT MACRO -->
-  <xacro:macro name="arctos_joint" params="name can_id gear_ratio limit_l limit_u" >
+  <xacro:macro name="arctos_joint" params="name can_id vel acc gear_ratio limit_l limit_u" >
     <joint name="${name}">
       <param name="can_id">${can_id}</param>
+      <param name="vel">${vel}</param>
+      <param name="acc">${acc}</param>
       <param name="gear_ratio">${gear_ratio}</param>
       <command_interface name="position">
@@ -31,16 +33,16 @@
           <class_type>arctos_hardware_interface::ArctosHardwareInterface</class_type>
           <param name="can_interface">can0</param>
-          <param name="accel">40</param>
-          <param name="vel">1000</param>
+          <!-- <param name="accel">20</param> -->
+          <!-- <param name="vel">500</param> -->
         </xacro:unless>
       </hardware>
       <!-- JOINT DEFINITIONS -->
-      <xacro:arctos_joint name="X_joint" can_id="1" gear_ratio="13.5" limit_l="${X_min_pos}" limit_u="${X_max_pos}"/>
-      <xacro:arctos_joint name="Y_joint" can_id="2" gear_ratio="-150.0" limit_l="${Y_min_pos}" limit_u="${Y_max_pos}"/>
-      <xacro:arctos_joint name="Z_joint" can_id="3" gear_ratio="150.0" limit_l="${Z_min_pos}" limit_u="${Z_max_pos}"/>
-      <xacro:arctos_joint name="A_joint" can_id="4" gear_ratio="48.0" limit_l="${A_min_pos}" limit_u="${A_max_pos}"/>
-      <xacro:arctos_joint name="B_joint" can_id="5" gear_ratio="67.82" limit_l="${B_min_pos}" limit_u="${B_max_pos}"/>
-      <xacro:arctos_joint name="C_joint" can_id="6" gear_ratio="67.82" limit_l="${C_min_pos}" limit_u="${C_max_pos}"/>
-      <xacro:arctos_joint name="Right_jaw_joint" can_id="7" gear_ratio="1" limit_l="0.0"
+      <xacro:arctos_joint name="X_joint" can_id="1" vel="1" acc="1.5" gear_ratio="13.5" limit_l="${X_min_pos}" limit_u="${X_max_pos}"/>
+      <xacro:arctos_joint name="Y_joint" can_id="2" vel="1" acc="3" gear_ratio="-150.0" limit_l="${Y_min_pos}" limit_u="${Y_max_pos}"/>
+      <xacro:arctos_joint name="Z_joint" can_id="3" vel="1" acc="3" gear_ratio="150.0" limit_l="${Z_min_pos}" limit_u="${Z_max_pos}"/>
+      <xacro:arctos_joint name="A_joint" can_id="4" vel="2" acc="8" gear_ratio="48.0" limit_l="${A_min_pos}" limit_u="${A_max_pos}"/>
+      <xacro:arctos_joint name="B_joint" can_id="5" vel="2" acc="8" gear_ratio="67.82" limit_l="${B_min_pos}" limit_u="${B_max_pos}"/>
+      <xacro:arctos_joint name="C_joint" can_id="6" vel="2" acc="8" gear_ratio="67.82" limit_l="${C_min_pos}" limit_u="${C_max_pos}"/>
+      <xacro:arctos_joint name="Right_jaw_joint" can_id="7" vel="3.5" acc='15.0' gear_ratio="1" limit_l="0.0"
       limit_u="0.015"/>
     <!-- </ros2_control>

Commit message: FIX: gripper open & close sync w/ moveit2 goal state

File: arctos_description/urdf/arctos.ros2_control.xacro (robot description, xacro)
@@ -3,4 +3,7 @@
   <!-- ARGUMENT TO TOGGLE FAKE HARDWARE -->
   <xacro:arg name="use_fake_hardware" default="false"/>
+  <!-- Gripper limits (shared for consistency) -->
+  <xacro:property name="gripper_limit_l" value="0.0"/>
+  <xacro:property name="gripper_limit_u" value="0.015"/>
   <!-- JOINT MACRO -->
   <xacro:macro name="arctos_joint" params="name can_id vel acc gear_ratio limit_l limit_u" >
@@ -33,4 +36,7 @@
           <class_type>arctos_hardware_interface::ArctosHardwareInterface</class_type>
           <param name="can_interface">can0</param>
+          <!-- Swap to invert gripper direction (easiest way) -->
+          <param name="gripper_open_position">${gripper_limit_u}</param>
+          <param name="gripper_close_position">${gripper_limit_l}</param>
           <!-- <param name="accel">20</param> -->
           <!-- <param name="vel">500</param> -->
@@ -44,6 +50,6 @@
       <xacro:arctos_joint name="B_joint" can_id="5" vel="2" acc="8" gear_ratio="67.82" limit_l="${B_min_pos}" limit_u="${B_max_pos}"/>
       <xacro:arctos_joint name="C_joint" can_id="6" vel="2" acc="8" gear_ratio="67.82" limit_l="${C_min_pos}" limit_u="${C_max_pos}"/>
-      <xacro:arctos_joint name="Right_jaw_joint" can_id="7" vel="3.5" acc='15.0' gear_ratio="1" limit_l="0.0"
-      limit_u="0.015"/>
+      <xacro:arctos_joint name="Right_jaw_joint" can_id="7" vel="3.5" acc='15.0' gear_ratio="1"
+      limit_l="${gripper_limit_l}" limit_u="${gripper_limit_u}"/>
     <!-- </ros2_control>
     <ros2_control name="gripper" type="system">

Commit message: add vel twist, pca, perception stack

File: arctos_description/urdf/arctos.ros2_control.xacro (robot description, xacro)
@@ -3,5 +3,5 @@
   <!-- ARGUMENT TO TOGGLE FAKE HARDWARE -->
   <xacro:arg name="use_fake_hardware" default="false"/>
-  <!-- Gripper limits (shared for consistency) -->
+  <!-- Gripper limits for the single actuated jaw; the left jaw mimics in the URDF. -->
   <xacro:property name="gripper_limit_l" value="0.0"/>
   <xacro:property name="gripper_limit_u" value="0.015"/>
@@ -36,5 +36,5 @@
           <class_type>arctos_hardware_interface::ArctosHardwareInterface</class_type>
           <param name="can_interface">can0</param>
-          <!-- Swap to invert gripper direction (easiest way) -->
+          <!-- Single-jaw gripper parameters consumed by ArctosHardwareInterface. -->
           <param name="gripper_open_position">${gripper_limit_u}</param>
           <param name="gripper_close_position">${gripper_limit_l}</param>
@@ -42,5 +42,5 @@
           <param name="wrist_roll_to_pitch_gain">0.0</param>
           <param name="wrist_b_feedback_gain">0.0</param>
-          <param name="wrist_c_feedback_gain">0.0</param>
+          <param name="wrist_c_feedback_gain">0.00</param>
           <!-- <param name="accel">20</param> -->
           <!-- <param name="vel">500</param> -->
@@ -54,23 +54,7 @@
       <xacro:arctos_joint name="B_joint" can_id="5" vel="2" acc="8" gear_ratio="67.82" limit_l="${B_min_pos}" limit_u="${B_max_pos}"/>
       <xacro:arctos_joint name="C_joint" can_id="6" vel="2" acc="8" gear_ratio="67.82" limit_l="${C_min_pos}" limit_u="${C_max_pos}"/>
-      <xacro:arctos_joint name="Right_jaw_joint" can_id="7" vel="3.5" acc='15.0' gear_ratio="1"
+      <!-- Only Right_jaw_joint is exported to ros2_control; Left_jaw_joint is a mimic joint. -->
+      <xacro:arctos_joint name="Right_jaw_joint" can_id="7" vel="3.5" acc="15.0" gear_ratio="1"
       limit_l="${gripper_limit_l}" limit_u="${gripper_limit_u}"/>
-    <!-- </ros2_control>
-    <ros2_control name="gripper" type="system">
-      <hardware>
-        <plugin>mock_components/GenericSystem</plugin>
-      </hardware> -->
-      <!-- <joint name="Right_jaw_joint">
-        <command_interface name="position"/>
-        <state_interface name="position">
-          <param name="initial_value">0.0</param>
-        </state_interface>
-        <state_interface name="velocity">
-          <param name="initial_value">0.0</param>
-        </state_interface>
-        <state_interface name="effort">
-          <param name="initial_value">0.0</param>
-        </state_interface>
-      </joint> -->
     </ros2_control>
   </xacro:macro>
