Commit message: amend: add mks sync mode and config mks drive(canid 6 for now) in on_config. change joint b&c revolute frm continous on urdf

File: arctos_moveit_config/arctos.urdf (robot description, URDF)
Before this commit: robot arctos, 12 links, 11 joints
Joints:
- joint A_joint: type continuous -> revolute
- joint B_joint: type continuous -> revolute
- joint C_joint: type continuous -> revolute
